File: Hardware/NTUT-PC104_16bit_64-40connectors_20250326-2025-03-31_v2/NTUT-PC104_16bit_64-40connectors_20250326-2025-03-31_v2.kicad_sch (KiCad schematic)
At the start: 41 parts, among them J10 Conn_02x26_Odd_Even, J12 Conn_02x04_Odd_Even, J13 Conn_02x04_Odd_Even, J14 Conn_02x04_Odd_Even, J15 Conn_02x04_Odd_Even, J16 Conn_02x04_Odd_Even, J17 Conn_02x04_Odd_Even, J18 Conn_02x04_Odd_Even, J7 Conn_02x04_Odd_Even, J8 Conn_02x26_Odd_Even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

Commit message: 1. Add power zones to associated pins on Left-up module. 2. Correct net names, i.e., upper/lower cases of net names.
Connections:
- net 5V_S-BAND_12W: now also J1.B5, J1.B6, J2.B5, J2.B6, J3.B5, J3.B6, J4.B5, J4.B6, J5.B5, J5.B6, J6.B5, J6.B6
- net 5V_S-Band_12W: no longer J1.B5, J1.B6, J2.B5, J2.B6, J3.B5, J3.B6, J4.B5, J4.B6, J5.B5, J5.B6, J6.B5, J6.B6
- net 5V_TT&C(UHF)_3.5W: now also J13.2 (Pin_2), J13.4 (Pin_4); no longer J13.6 (Pin_6), J13.8 (Pin_8)
- net 5V_TT&C(VHF)_3.5W: now also J13.6 (Pin_6), J13.8 (Pin_8); no longer J13.2 (Pin_2), J13.4 (Pin_4)
- now unconnected: J17.2 (Pin_2), J17.4 (Pin_4), J17.6 (Pin_6), J17.8 (Pin_8)
- no-connect marks 2 -> 5
Changed lines of the file:
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@@
 	)
 	(junction
-		(at 554.99 344.17)
-		(diameter 0)
-		(color 0 0 0 0)
-	)
-	(junction
 		(at 534.67 278.13)
 		(diameter 0)
@@
 	)
 	(junction
-		(at 554.99 341.63)
-		(diameter 0)
-		(color 0 0 0 0)
-	)
-	(junction
 		(at 534.67 355.6)
 		(diameter 0)
@@
 	)
 	(junction
-		(at 554.99 339.09)
-		(diameter 0)
-		(color 0 0 0 0)
-	)
-	(junction
 		(at 534.67 289.56)
 		(diameter 0)
@@
 	)
 	(no_connect
+		(at 554.99 344.17)
+	)
+	(no_connect
+		(at 554.99 339.09)
+	)
+	(no_connect
 		(at 632.46 -85.09)
 	)
 	(no_connect
-		(at 560.07 339.09)
+		(at 554.99 346.71)
+	)
+	(no_connect
+		(at 554.99 341.63)
 	)
 	(wire
@@
 	(wire
 		(pts
-			(xy 554.99 346.71) (xy 554.99 344.17)
-		)
-		(stroke
-			(width 0)
-			(type default)
-		)
-	)
-	(wire
-		(pts
 			(xy 113.03 149.86) (xy 132.08 149.86)
 		)
@@
 	(wire
 		(pts
-			(xy 554.99 341.63) (xy 554.99 339.09)
-		)
-		(stroke
-			(width 0)
-			(type default)
-		)
-	)
-	(wire
-		(pts
 			(xy 158.75 294.64) (xy 181.61 294.64)
 		)
@@
 	(wire
 		(pts
-			(xy 549.91 339.09) (xy 554.99 339.09)
-		)
-		(stroke
-			(width 0)
-			(type default)
-		)
-	)
-	(wire
-		(pts
 			(xy 549.91 278.13) (xy 554.99 278.13)
 		)
@@
 	(wire
 		(pts
-			(xy 30.48 71.12) (xy 49.53 71.12)
+			(xy 549.91 339.09) (xy 554.99 339.09)
 		)
 		(stroke
@@
 	(wire
 		(pts
-			(xy 405.13 48.26) (xy 424.18 48.26)
+			(xy 30.48 71.12) (xy 49.53 71.12)
 		)
 		(stroke
@@
 	(wire
 		(pts
-			(xy 549.91 280.67) (xy 554.99 280.67)
+			(xy 405.13 48.26) (xy 424.18 48.26)
 		)
 		(stroke
@@
 	(wire
 		(pts
-			(xy 537.21 264.16) (xy 534.67 264.16)
+			(xy 549.91 280.67) (xy 554.99 280.67)
 		)
 		(stroke
@@
 	(wire
 		(pts
-			(xy 276.86 86.36) (xy 295.91 86.36)
+			(xy 537.21 264.16) (xy 534.67 264.16)
 		)
 		(stroke
@@
 	(wire
 		(pts
-			(xy 405.13 157.48) (xy 424.18 157.48)
+			(xy 276.86 86.36) (xy 295.91 86.36)
 		)
 		(stroke
@@
 	(wire
 		(pts
-			(xy 549.91 297.18) (xy 554.99 297.18)
+			(xy 405.13 157.48) (xy 424.18 157.48)
 		)
 		(stroke
@@
 	(wire
 		(pts
-			(xy 534.67 246.38) (xy 534.67 243.84)
+			(xy 549.91 297.18) (xy 554.99 297.18)
 		)
 		(stroke
@@
 	(wire
 		(pts
-			(xy 554.99 339.09) (xy 560.07 339.09)
+			(xy 534.67 246.38) (xy 534.67 243.84)
 		)
 		(stroke
@@
 	(wire
 		(pts
-			(xy 554.99 344.17) (xy 554.99 341.63)
-		)
-		(stroke
-			(width 0)
-			(type default)
-		)
-	)
-	(wire
-		(pts
 			(xy 438.15 60.96) (xy 457.2 60.96)
 		)
@@
 		)
 	)
-	(label "5V_S-Band_12W"
+	(label "5V_S-BAND_12W"
 		(at 327.66 45.72 0)
 		(effects
@@
 		)
 	)
-	(label "5V_S-Band_12W"
+	(label "5V_S-BAND_12W"
 		(at 488.95 48.26 0)
 		(effects
@@
 		)
 	)
-	(label "5V_S-Band_12W"
+	(label "5V_S-BAND_12W"
 		(at 81.28 48.26 0)
 		(effects
@@
 		)
 	)
-	(label "5V_S-Band_12W"
+	(label "5V_S-BAND_12W"
 		(at 488.95 45.72 0)
 		(effects
@@
 		)
 	)
-	(label "5V_TT&C(VHF)_3.5W"
-		(at 556.26 273.05 0)
-		(effects
-			(font
-				(size 1.27 1.27)
-			)
-			(justify left bottom)
-		)
-	)
 	(label "5V_ADCS_1.2W"
 		(at 163.83 274.32 0)
@@
 		)
 	)
-	(label "5V_S-Band_12W"
+	(label "5V_S-BAND_12W"
 		(at 163.83 45.72 0)
 		(effects
@@
 		)
 	)
-	(label "5V_TPM_0.4W"
-		(at 556.26 355.6 0)
-		(effects
-			(font
-				(size 1.27 1.27)
-				(color 255 0 30 1)
-			)
-			(justify left bottom)
-		)
-	)
 	(label "OUTPW4"
 		(at 438.15 78.74 0)
@@
 		)
 	)
-	(label "5V_S-Band_12W"
+	(label "5V_S-BAND_12W"
 		(at 81.28 45.72 0)
 		(effects
@@
 		)
 	)
-	(label "5V_S-Band_12W"
+	(label "5V_S-BAND_12W"
 		(at 245.11 48.26 0)
 		(effects
@@
 		)
 	)
+	(label "5V_TT&C(UHF)_3.5W"
+		(at 557.53 273.05 0)
+		(effects
+			(font
+				(size 1.27 1.27)
+			)
+			(justify left bottom)
+		)
+	)
 	(label "PPS"
 		(at 163.83 251.46 0)
@@
 		)
 	)
+	(label "5V_GPSR_0.6W"
+		(at 560.07 360.68 0)
+		(effects
+			(font
+				(size 1.27 1.27)
+			)
+			(justify left bottom)
+		)
+	)
 	(label "GND"
 		(at 194.31 35.56 0)
@@
 		)
 	)
+	(label "5V_TT&C(VHF)_3.5W"
+		(at 557.53 278.13 0)
+		(effects
+			(font
+				(size 1.27 1.27)
+			)
+			(justify left bottom)
+		)
+	)
 	(label "D7"
 		(at 488.95 139.7 0)
@@
 		)
 	)
-	(label "5V_S-Band_12W"
+	(label "5V_S-BAND_12W"
 		(at 245.11 45.72 0)
 		(effects
@@
 		)
 	)
-	(label "5V_S-Band_12W"
+	(label "5V_S-BAND_12W"
 		(at 327.66 48.26 0)
 		(effects
@@
 		)
 	)
-	(label "5V_TT&C(UHF)_3.5W"
-		(at 556.26 278.13 0)
-		(effects
-			(font
-				(size 1.27 1.27)
-			)
-			(justify left bottom)
-		)
-	)
 	(label "OUTPW2"
 		(at 113.03 83.82 0)
@@
 		)
 	)
-	(label "5V_S-Band_12W"
+	(label "5V_S-BAND_12W"
 		(at 406.4 45.72 0)
 		(effects
@@
 		)
 	)
+	(label "5V_TPM_0.4W"
+		(at 560.07 355.6 0)
+		(effects
+			(font
+				(size 1.27 1.27)
+				(color 255 0 30 1)
+			)
+			(justify left bottom)
+		)
+	)
 	(label "GND"
 		(at 488.95 63.5 0)
@@
 		)
 	)
-	(label "5V_S-Band_12W"
+	(label "5V_S-BAND_12W"
 		(at 406.4 48.26 0)
 		(effects
@@
 		)
 	)
-	(label "5V_GPSR_0.6W"
-		(at 556.26 360.68 0)
-		(effects
-			(font
-				(size 1.27 1.27)
-			)
-			(justify left bottom)
-		)
-	)
 	(label "C19"
 		(at 257.81 349.25 0)
@@
 		)
 	)
-	(label "5V_S-Band_12W"
+	(label "5V_S-BAND_12W"
 		(at 163.83 48.26 0)
 		(effects

Commit message: 1. All power zones added.
Connections:
- net 5V_S-BAND_12W: now also J9.10 (Pin_10), J9.12 (Pin_12), JA19.10 (Pin_10), JA19.12 (Pin_12)
- net 5V_S-Band_12W: no longer J9.10 (Pin_10), J9.12 (Pin_12), JA19.10 (Pin_10), JA19.12 (Pin_12)
- no-connect marks 5 -> 4
