File: Hardware/NTUT-PC104_16bit_64-40connectors_2025-05-07_v4.1/NTUT-PC104_16bit_64-40connectors_2025-05-07_v4.1.kicad_pcb (KiCad board)
At the start: 4 copper layers, 390.3 x 285.7 mm, 51 parts, among them J10 Conn_02x26_Odd_Even, J12 Conn_02x04_Odd_Even, J13 Conn_02x04_Odd_Even, J14 Conn_02x04_Odd_Even, J15 Conn_02x04_Odd_Even, J16 Conn_02x04_Odd_Even, J17 Conn_02x04_Odd_Even, J18 Conn_02x04_Odd_Even, J19 Conn_01x04, J20 Conn_01x04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

Commit message: Add a new PCB view image file.
Other:
- board text removed: "${FILENAME}"
Changed lines of the file:
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@@
-		)
-	)
-	(gr_text "${FILENAME}"
-		(at 187.458398 111.887 0)
-		(layer "F.SilkS")
-		(effects
-			(font
-				(size 1 1)
-				(thickness 0.15)
-			)
-			(justify left bottom)
 		)
 	)
